File: pcb/neighboard-plate.kicad_pcb (KiCad board)
At the start: 2 copper layers, 279.8 x 96 mm, 30 parts, among them SW1 Switch, SW10 Switch, SW11 Switch, SW12 Switch, SW13 Switch, SW14 Switch, SW15 Switch, SW16 Switch, SW17 Switch, SW18 Switch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

Commit message: Add Ground Fill
Routing:
- net (no net): track 0.00 -> 10.0 mm
- added copper zone on B.Cu, net (none)
- added copper zone on F.Cu, net (none)
Changed lines of the file:
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@@
       (xy 89.932306 49.886409)
     )
-    (stroke (width 0) (type solid)) (fill none) (layer "Edge.Cuts"))
+    (stroke (width 0.1) (type solid)) (fill none) (layer "Edge.Cuts"))
   (gr_poly
     (pts
@@
     )
     (stroke (width 0.1) (type solid)) (fill none) (layer "Edge.Cuts"))
+  (segment (start 223 83) (end 227 83) (width 0.25) (layer "B.Cu") (net 0))
+  (segment (start 80 84) (end 86 84) (width 0.25) (layer "B.Cu") (net 0))
+  (zone (net 0) (net_name "") (layers "F&B.Cu") (hatch edge 0.5)
+    (connect_pads (clearance 0.5))
+    (min_thickness 0.25) (filled_areas_thickness no)
+    (fill yes (thermal_gap 0.5) (thermal_bridge_width 0.5) (island_removal_mode 1) (island_area_min 10))
+    (polygon
+      (pts
+        (xy 7 38)
+        (xy 311 38)
+        (xy 311 165)
+        (xy 7 165)
+      )
+    )
+  )
   (group "" (id 8b8978ee-839a-4507-9320-d6914aed99f0)
     (members

Commit message: Add Mounting Holes
Parts:
- added Ref**: Val**, footprints:m2-hole, F.Cu at (287.3, 119.8)
- added Ref**: Val**, footprints:m2-hole, F.Cu at (76.7, 126.7)
- added Ref**: Val**, footprints:m2-hole, F.Cu at (145.9, 98.0)
- added Ref**: Val**, footprints:m2-hole, F.Cu at (337.1, 126.2)
- added Ref**: Val**, footprints:m2-hole, F.Cu at (126.4, 120.2)
- added Ref**: Val**, footprints:m2-hole, F.Cu at (192.5, 155.8)
- added Ref**: Val**, footprints:m2-hole, F.Cu at (267.8, 97.5)
- added Ref**: Val**, footprints:m2-hole, F.Cu at (221.2, 155.4)
- moved SW17 63.5 mm to (277.9, 94.2)
- moved SW27 63.5 mm to (296.6, 135.7)
- moved SW4 63.5 mm to (94.4, 135.2)
- moved SW16 63.5 mm to (257.8, 101.0)
- moved SW20 63.5 mm to (258.4, 118.0)
- moved SW22 63.5 mm to (297.2, 118.7)
- moved SW10 63.5 mm to (117.1, 136.2)
- moved SW14 63.5 mm to (173.5, 161.1)
- moved SW3 63.5 mm to (155.8, 101.5)
- moved SW5 63.5 mm to (116.5, 119.2)
- moved SW6 63.5 mm to (135.8, 111.7)
- moved SW8 63.5 mm to (173.4, 114.9)
- moved SW1 63.5 mm to (115.9, 102.2)
- moved SW11 63.5 mm to (135.8, 128.7)
- moved SW15 63.5 mm to (190.0, 165.5)
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
Commit message: Scratch work
Other:
- board size 279.8 x 96 mm -> 283.9 x 99.9 mm
