File: pcb/neighboard.kicad_pcb (KiCad board)
At the start: 2 copper layers, 281.5 x 95.9 mm, 72 parts, among them SW1 Switch, SW10 Switch, SW11 Switch, SW12 Switch, SW13 Switch, SW14 Switch, SW15 Switch, SW16 Switch, SW17 Switch, SW18 Switch, SW19 Switch, SW2 Switch, SW20 Switch, SW21 Switch, SW22 Switch, SW23 Switch, SW24 Switch, SW25 Switch, SW26 Switch, SW27 Switch, SW28 Switch, SW29 Switch, SW3 Switch, SW30 Switch, SW31 SW_SPDT, SW32 SW_SPDT, SW33 SW_Push, SW34 SW_Push, SW4 Switch, SW5 Switch, SW6 Switch, SW7 Switch, SW8 Switch, SW9 Switch, U1 xiao-ble, U2 xiao-ble

Commit message: Add Ground Fill
Routing:
- added copper zone on B.Cu, net GND L
- added copper zone on F.Cu, net GND L
Changed lines of the file:
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@@
   (segment (start 255.943321 139.466123) (end 229.193321 139.466123) (width 0.25) (layer "B.Cu") (net 65))
   (segment (start 227.993321 138.266123) (end 223.879047 138.266123) (width 0.25) (layer "B.Cu") (net 65))
+  (zone (net 2) (net_name "GND L") (layers "F&B.Cu") (hatch edge 0.5)
+    (connect_pads (clearance 0))
+    (min_thickness 0.25) (filled_areas_thickness no)
+    (fill yes (thermal_gap 0.5) (thermal_bridge_width 0.5) (island_removal_mode 2) (island_area_min 2))
+    (polygon
+      (pts
+        (xy 60.5 84.5)
+        (xy 367 84.5)
+        (xy 367 221.5)
+        (xy 60.5 221.5)
+      )
+    )
+  )
   (group "" (id 57188aed-87e3-4d8f-bc8a-8f4aac7fce00)
     (members

Commit message: Add Mounting Holes
Parts:
- added Ref**: Val**, footprints:m2-hole, F.Cu at (228.8, 145.9)
- added Ref**: Val**, footprints:m2-hole, F.Cu at (85.1, 142.8)
- added Ref**: Val**, footprints:m2-hole, F.Cu at (134.9, 136.3)
- added Ref**: Val**, footprints:m2-hole, F.Cu at (154.4, 114.0)
- added Ref**: Val**, footprints:m2-hole, F.Cu at (295.9, 135.8)
- added Ref**: Val**, footprints:m2-hole, F.Cu at (201.0, 171.9)
- added Ref**: Val**, footprints:m2-hole, F.Cu at (345.6, 142.3)
- added Ref**: Val**, footprints:m2-hole, F.Cu at (229.8, 171.5)
- added Ref**: Val**, footprints:m2-hole, F.Cu at (201.9, 146.4)
- added Ref**: Val**, footprints:m2-hole, F.Cu at (276.3, 113.6)
Routing:
- net Row2L: track 120.1 -> 122.8 mm
- net Row1L: track 106.1 -> 104.8 mm
- net Bat+ L: track 137.5 -> 136.2 mm
- net GND L: track 126.4 -> 127.2 mm

Commit message: Scratch work
Parts:
- removed the Ref** at (228.8, 145.9)
- removed the Ref** at (85.1, 142.8)
- removed the Ref** at (134.9, 136.3)
- removed the Ref** at (154.4, 114.0)
- removed the Ref** at (295.9, 135.8)
- removed the Ref** at (201.0, 171.9)
- removed the Ref** at (345.6, 142.3)
- removed the Ref** at (229.8, 171.5)
- removed the Ref** at (201.9, 146.4)
- removed the Ref** at (276.3, 113.6)
- added Ref**: Val**, footprints:m2-hole, F.Cu at (124.0, 130.2)
- added Ref**: Val**, footprints:m2-hole, F.Cu at (223.3, 139.3)
- added Ref**: Val**, footprints:m2-hole, F.Cu at (143.5, 108.0)
- added Ref**: Val**, footprints:m2-hole, F.Cu at (190.1, 165.8)
- added Ref**: Val**, footprints:m2-hole, F.Cu at (272.8, 107.5)
- added Ref**: Val**, footprints:m2-hole, F.Cu at (342.1, 136.3)
- added Ref**: Val**, footprints:m2-hole, F.Cu at (226.3, 165.4)
- added Ref**: Val**, footprints:m2-hole, F.Cu at (193.1, 139.7)
- added Ref**: Val**, footprints:m2-hole, F.Cu at (292.4, 129.7)
- added Ref**: Val**, footprints:m2-hole, F.Cu at (74.2, 136.7)
- moved BT1 16.9 mm to (80.9, 114.3)
- moved D8 12.5 mm to (171.2, 120.1)
- moved SW13 12.5 mm to (170.4, 141.8)
- moved D13 12.5 mm to (170.6, 137.1)
- moved SW14 12.5 mm to (171.1, 171.1)
- moved SW5 12.5 mm to (114.1, 129.1)
- moved D12 12.5 mm to (152.4, 140.7)
- moved SW2 12.5 mm to (133.4, 104.6)
- moved D11 12.5 mm to (133.4, 133.9)
- moved D10 12.5 mm to (114.5, 141.4)
- moved D14 12.5 mm to (174.6, 172.3)
- moved D4 12.5 mm to (87.3, 145.5)
- moved SW7 12.5 mm to (152.9, 128.4)
- moved D6 12.5 mm to (133.4, 116.9)
- moved SW1 12.5 mm to (113.5, 112.1)
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Routing:
- net Row4R: track 51.8 -> 63.2 mm, vias 1 -> 0
- net Bat+ L: track 136.2 -> 125.9 mm
- net ResetL: track 60.5 -> 70.0 mm
- net Bat- R: track 188.2 -> 178.8 mm, vias 2 -> 4
- net ResetR: track 73.5 -> 81.9 mm
- net GND L: track 127.2 -> 119.0 mm, vias 7 -> 2
- net Col5R: track 96.8 -> 104.4 mm, vias 2 -> 0
- net Bat- L: track 181.9 -> 189.5 mm
- net Row2L: track 122.8 -> 128.6 mm
- net Col5L: track 82.1 -> 86.2 mm, vias 1 -> 3
- net Col1R: track 152.8 -> 156.0 mm
- net Col4R: track 126.3 -> 129.1 mm
- net Col2R: track 132.1 -> 134.6 mm
- net Col1L: track 133.9 -> 136.2 mm, vias 1 -> 3
- net Row3L: track 129.8 -> 132.1 mm
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Other:
- board size 281.5 x 95.9 mm -> 295.3 x 99.9 mm
